Commit message: Delete unnecesary transformation

File: zed_wrapper/urdf/zed_macro.urdf.xacro (robot description, xacro)
@@ -88,10 +88,4 @@
       <origin xyz="0 ${baseline/2} 0" rpy="0 0 0" />
     </joint>
-    <link name="${name}_left_camera_optical_frame"/>
-    <joint name="${name}_left_camera_optical_joint" type="fixed">
-      <origin xyz="${optical_offset_x} 0 0" rpy="-${M_PI/2} 0.0 -${M_PI/2}"/>
-      <parent link="${name}_left_camera_frame"/>
-      <child link="${name}_left_camera_optical_frame"/>
-    </joint>
     <!-- Right Camera -->
     <link name="${name}_right_camera_frame" />
@@ -100,10 +94,4 @@
       <child link="${name}_right_camera_frame"/>
       <origin xyz="0 -${baseline/2} 0" rpy="0 0 0" />
-    </joint>
-    <link name="${name}_right_camera_optical_frame"/>
-    <joint name="${name}_right_camera_optical_joint" type="fixed">
-      <origin xyz="${optical_offset_x} 0 0" rpy="-${M_PI/2} 0.0 -${M_PI/2}"/>
-      <parent link="${name}_right_camera_frame"/>
-      <child link="${name}_right_camera_optical_frame"/>
     </joint>
     <!-- ZED2 Sensors -->
